Commit message: Commit 10/5 -Modificaciones en el CMakelist. -Añadidos parametros en rviz para que utilice el tiempo del simulador. -Añadido el subscriptor del Lidar y los metodos para esquivar obstaculos, con transicion de estados y la acción de estados. Cambiada la forma de moverse del dron para que el morro siempre apunte hacia el frente. -Cambiados waypoints en el Controller_node y umbrales de seguridad en el security_node -Modificado el URDF del dron para añadir una nariz roja en el frontal para saber cual es el morro del dron.

File: src/drone_control/urdf/drone.urdf.xacro (robot description, xacro)
@@ -3,4 +3,7 @@
     <material name="blue">
         <color rgba="0 0 0.8 1"/>
+    </material>
+    <material name="red">
+        <color rgba="0.8 0 0 1"/>
     </material>
     <material name="black">
@@ -32,8 +35,23 @@
         </inertial>
     </link>
+    <joint name="nose_joint" type="fixed">
+        <parent link="chassis"/>
+        <child link="nose_link"/>
+        <origin xyz="0.2 0 0.0" rpy="0 0 0"/>
+    </joint>
+    <link name="nose_link">
+        <visual>
+            <origin xyz="0 0 0" rpy="0 0 0"/>
+            <geometry>
+                <box size="0.1 0.1 0.05"/>
+            </geometry>
+            <material name = "red"/>
+        </visual>
+    </link>
     <joint name="lidar_joint" type="fixed">
         <parent link="chassis"/>
         <child link="lidar_link"/>
-        <origin xyz="0 0 0.075" rpy="0 0 0"/> </joint>
+        <origin xyz="0 0 0.075" rpy="0 0 0"/>
+    </joint>
     <link name="lidar_link">
         <visual>
@@ -65,8 +83,9 @@
     <!-- PLUGIN DE GAZEBO: SENSOR LIDAR                 -->
     <!-- ============================================== -->
-    <gazebo reference="lidar_link">
+    <gazebo reference="base_link">
         <sensor name="lidar" type="gpu_lidar">
+            <pose>0 0 0.075 0 0 0</pose>
             <topic>/scan</topic>
-            <gz_frame_id>lidar_link</gz_frame_id>
+            <gz_frame_id>base_link</gz_frame_id>
             <update_rate>10</update_rate> <!-- Lee datos a 10 Hz -->
             <ray>
@@ -91,5 +110,5 @@
             </ray>
             <always_on>true</always_on><!-- poner a false para no ver los rayos-->
-            <visualize>true</visualize>
+            <visualize>false</visualize>
         </sensor>
     </gazebo>
@@ -99,4 +118,5 @@
         <plugin filename="libgz-sim-velocity-control-system.so" name="gz::sim::systems::VelocityControl">
             <topic>/cmd_vel</topic>
+            <use_world_frame>false</use_world_frame>
         </plugin>
         <!-- 2. El "GPS": Publica la Odometría para saber dónde está el dron -->
